File: 3.5_SAS_Backend.kicad_pcb (KiCad board)
At the start: 2 copper layers, 86.4 x 97.2 mm, 30 parts, among them M2 MountingHole_2.2mm_M2, M3 MountingHole_3.2mm_M3, SW1 SW_DIP_x01, U1 ZXDN10_S1205SAW, U2 DC_022B_5.5*2.1_2, U3 DC_022B_5.5*2.1_2, U4 SAS_29, U5 SAS_29, U6 SAS_29, U7 SAS_29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

Commit message: fix bugs
Parts:
- moved M3 12.7 mm to (80.6, 48.3)
- moved ADJ_FAN 6.99 mm to (80.6, 41.9)
- moved C3 1.91 mm to (92.1, 61.6)
- moved M3 0.64 mm to (80.6, 125.7)
Routing:
- net GND: track 428.8 -> 449.3 mm
- net +5V: track 458.8 -> 463.8 mm
- net Net-(M3-Pad2): track 23.9 -> 26.3 mm
